File: 01_power_management.kicad_sch (KiCad schematic)
At the start: 37 parts, among them Q1 AO3401A, SW1 K3-1296S-J1, U1 XDJK-0051-025, U2 LM66100DCKR, U3 LM66100DCKR, U4 AP63205WU-7, U5 USBLC6-2SC6, U7 AP2112K-3.3TRG1

Commit message: Update on the CE pad from the component U2
Connections:
- net GND: now also U2.3 (~{CE})
- net USBVCC: no longer U2.3 (~{CE})
Changed lines of the file:
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@@
+	)
+	(junction
+		(at 154.94 33.02)
+		(diameter 0)
+		(color 0 0 0 0)
 	)
 	(junction
@@
 	(junction
 		(at 255.27 29.21)
-		(diameter 0)
-		(color 0 0 0 0)
-	)
-	(junction
-		(at 154.94 50.8)
 		(diameter 0)
 		(color 0 0 0 0)
@@
 	(wire
 		(pts
-			(xy 149.86 50.8) (xy 154.94 50.8)
+			(xy 149.86 50.8) (xy 156.21 50.8)
 		)
 		(stroke
@@
 	(wire
 		(pts
-			(xy 149.86 33.02) (xy 156.21 33.02)
+			(xy 149.86 33.02) (xy 154.94 33.02)
 		)
 		(stroke
@@
 	(wire
 		(pts
+			(xy 154.94 33.02) (xy 156.21 33.02)
+		)
+		(stroke
+			(width 0)
+			(type default)
+		)
+	)
+	(wire
+		(pts
 			(xy 53.34 38.1) (xy 53.34 43.18)
 		)
@@
 	(wire
 		(pts
-			(xy 154.94 35.56) (xy 154.94 50.8)
-		)
-		(stroke
-			(width 0)
-			(type default)
-		)
-	)
-	(wire
-		(pts
 			(xy 220.98 31.75) (xy 224.79 31.75)
 		)
@@
 	(wire
 		(pts
+			(xy 154.94 33.02) (xy 154.94 35.56)
+		)
+		(stroke
+			(width 0)
+			(type default)
+		)
+	)
+	(wire
+		(pts
 			(xy 34.29 45.72) (xy 34.29 43.18)
 		)
@@
 		)
 		(stroke
-			(width 0)
-			(type default)
-		)
-	)
-	(wire
-		(pts
-			(xy 154.94 50.8) (xy 156.21 50.8)
-		)
-		(stroke
