File: arduino_uno.kicad_pcb (KiCad board)
At the start: 2 copper layers, 53.3 x 68.6 mm, 85 parts, among them J1 ICSP1 Header, J10 GND Header, J2 Analog GPIO Header, J3 Numeric/Analog GPIO Header 2, J4 Numeric GPIO Header, J5 Power Header, J6 Numeric/Analog GPIO Header 1, J7 I2C Header, J8 UART Header, J9 Power Output Header, Q1 AO3401A, SW1 K3-1296S-J1, SW2 PTS526SM15SMTR2LFS, U1 XDJK-0051-025, U2 LM66100DCKR, U3 LM66100DCKR, U4 AP63205WU-7, U5 USBLC6-2SC6, U6 CH9101R, U7 AP2112K-3.3TRG1, U8 ATMEGA328PB-MN, X1 STD-CSW-5

Commit message: Update on the CE pad from the component U2
Connections:
- U2 pad 3: USBVCC -> GND
Routing:
- net USBVCC: track 35.9 -> 35.1 mm
- net GND: vias 173 -> 174
Changed lines of the file:
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@@
 			(size 0.35 0.85)
 			(layers "F.Cu" "F.Mask" "F.Paste")
-			(net "USBVCC")
+			(net "GND")
 			(pinfunction "~{CE}_3")
 			(pintype "unspecified")
@@
 	)
 	(via
-		(at 122 68)
+		(at 122.03 68.09)
 		(size 0.6)
 		(drill 0.25)
@@
 	)
 	(via
+		(at 123.02 68.15)
+		(size 0.6)
+		(drill 0.25)
+		(layers "F.Cu" "B.Cu")
+		(free yes)
+		(net "GND")
+	)
+	(via
 		(at 149.593 108.715)
 		(size 0.6)
@@
 	)
 	(segment
-		(start 123.155 71.31)
-		(end 123.155 68.935)
+		(start 147.49 63.54)
+		(end 147.5 63.55)
 		(width 0.25)
 		(layer "F.Cu")
@@
 	)
 	(segment
-		(start 147.49 63.54)
-		(end 147.5 63.55)
+		(start 123.8 68.86)
+		(end 123.81 68.85)
 		(width 0.25)
 		(layer "F.Cu")
@@
 	)
 	(segment
-		(start 124.1 72.255)
-		(end 123.155 71.31)
+		(start 123.28 69.12)
+		(end 123.54 68.86)
 		(width 0.25)
 		(layer "F.Cu")
@@
 	)
 	(segment
-		(start 123.155 68.935)
-		(end 123.23 68.86)
+		(start 123.54 68.86)
+		(end 123.8 68.86)
 		(width 0.25)
 		(layer "F.Cu")
@@
 	)
 	(segment
-		(start 140.03 66.56)
-		(end 140.64 65.95)
+		(start 123.28 70.11599)
+		(end 123.28 69.12)
 		(width 0.25)
 		(layer "F.Cu")
@@
 	)
 	(segment
-		(start 123.8 68.86)
-		(end 123.81 68.85)
+		(start 140.03 66.56)
+		(end 140.64 65.95)
 		(width 0.25)
 		(layer "F.Cu")
@@
 	)
 	(segment
-		(start 123.23 68.86)
-		(end 123.8 68.86)
+		(start 132.71 73.33)
+		(end 124.59 73.33)
 		(width 0.25)
 		(layer "F.Cu")
@@
 	)
 	(segment
-		(start 122.68 68.86)
-		(end 123.23 68.86)
+		(start 135.345 70.53)
+		(end 135.345 71.695)
 		(width 0.25)
 		(layer "F.Cu")
@@
 	)
 	(segment
-		(start 135.345 70.53)
-		(end 135.345 71.695)
+		(start 124.59 73.33)
+		(end 124.1 72.84)
 		(width 0.25)
 		(layer "F.Cu")
@@
 	)
 	(segment
-		(start 124.59 73.33)
-		(end 124.1 72.84)
+		(start 124.1 72.255)
+		(end 123.155 71.31)
 		(width 0.25)
 		(layer "F.Cu")
@@
 	)
 	(segment
-		(start 132.71 73.33)
-		(end 124.59 73.33)
+		(start 123.155 71.31)
+		(end 123.155 70.24099)
+		(width 0.25)
+		(layer "F.Cu")
+		(net "USBVCC")
+	)
+	(segment
+		(start 123.155 70.24099)
+		(end 123.28 70.11599)
 		(width 0.25)
 		(layer "F.Cu")
